Commit message: `cd external/bullet3 && git pull`.

File: external/bullet3/examples/pybullet/gym/pybullet_data/a1/a1.urdf (robot description, URDF)
Before this commit: robot a1_description, 22 links, 21 joints
Links:
- link FL_upper_shoulder: mass None -> 0.001
- link FR_upper_shoulder: mass None -> 0.001
- link RL_upper_shoulder: mass None -> 0.001
- link RR_upper_shoulder: mass None -> 0.001
